File: FPGA/doc/up_down_counter/up_down_counter.kicad_sch (KiCad schematic)
At the start: 6 parts

Commit message: 0219 work upload
Connections:
- new net: u_fnd_digit_display1. (seg), u_fnd_digit_select1. (sel)
- new net: u_bin2bcd4digit1. (digit1000_3:0), u_fnd_digit_display1. (seg) (x4)
Other:
- note added: "mux가 더 맞음"
Changed lines of the file:
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@@
+		)
+	)
+	(text "mux가 더 맞음"
+		(exclude_from_sim no)
+		(at 84.328 103.632 0)
+		(effects
+			(font
+				(size 1.27 1.27)
+			)
 		)
 	)

Commit message: 0220 work upload
Parts:
- added u_blink1: blink, symbol debounce:u_blink
Connections:
- net seg_data_13:0 is gone; now on net seg_data_12:0: u_control_tower1. (seg_dat), u_fnd_controller1. (seg)
- net sw_7:0 is gone; now on net seg_data_12:0: u_control_tower1. (seg_dat)
- net clk: now also u_blink1. (seg_dot)
- net reset: now also u_blink1. (seg_dot)
- net seg_dot: now reaches u_fnd_digit_display1. (seg)
- net seg_dot: no longer u_fnd_digit_select1. (sel)
- net led_15:0 renamed seg_data_12:0
- new net: u_fnd_digit_display1. (seg), u_fnd_digit_select1. (idle_state) (x2)
- new net: u_bin2bcd4digit1. (digit1000_3:0), u_fnd_digit_display1. (seg) (x4)
- new net: u_blink1. (seg_dot), u_fnd_controller1. (seg)
- new net idle: u_control_tower1. (seg_dat), u_fnd_controller1. (seg), u_fnd_digit_display1. (seg), u_fnd_digit_select1. (idle_state)
Other:
- moved on the sheet: u_bin2bcd4digit1
